Commit message: Sync elfin_humble_ws to the current Humble workspace snapshot.
Bring the nested workspace up to the local packing/perception tree,
including the PF-R chain, agent mailbox contract, container hull tests,
and D555 bring-up dispatch, without replacing deployment_ws.

Co-authored-by: Cursor <cursoragent@cursor.com>

File: elfin_humble_ws/src/luggage_description/config/mid360_origin.xacro (robot description, xacro)
@@ -24,3 +24,15 @@
   <xacro:property name="livox_imu_xyz" value="0.01100 0.02329 -0.04412"/>
   <xacro:property name="livox_imu_rpy" value="0 0 0"/>
+  <!-- Sim gpu_lidar (repeating raster, not the real non-repetitive scan).
+       Handbook FOV 360° × (−7° … +52°); typical range 40 m @ 10% reflectivity.
+       Min 0.1 m matches the close-range blind zone. -->
+  <xacro:property name="livox_sim_update_hz" value="10.0"/>
+  <xacro:property name="livox_sim_h_samples" value="360"/>
+  <xacro:property name="livox_sim_v_samples" value="32"/>
+  <xacro:property name="livox_sim_h_min" value="-3.14159265"/>
+  <xacro:property name="livox_sim_h_max" value="3.14159265"/>
+  <xacro:property name="livox_sim_v_min" value="-0.12217305"/>
+  <xacro:property name="livox_sim_v_max" value="0.90757121"/>
+  <xacro:property name="livox_sim_range_min" value="0.1"/>
+  <xacro:property name="livox_sim_range_max" value="40.0"/>
 </robot>

File: elfin_humble_ws/src/luggage_description/urdf/eef_sensor_mount.urdf.xacro (robot description, xacro)
@@ -44,5 +44,8 @@
          xyz/rpy are the camera-tower +Y pad, not jointly calibrated). -->
     <link name="mid360_mount_frame">
-      <!-- Housing 65 x 65 x 60 mm, origin at base centre, +Z through the dome. -->
+      <!-- Housing 65 x 65 x 60 mm, origin at base centre, +Z through the dome.
+           Visual only: a collision mesh at the optical origin would fill a
+           360° gpu_lidar with self-hits. Range min 0.1 m already covers the
+           60 mm body. -->
       <visual>
         <origin xyz="0 0 0.030" rpy="0 0 0"/>
@@ -54,4 +57,11 @@
         </material>
       </visual>
+      <inertial>
+        <mass value="0.265"/>
+        <origin xyz="0 0 0.030" rpy="0 0 0"/>
+        <inertia ixx="0.000180" ixy="0.0" ixz="0.0"
+                 iyy="0.000180" iyz="0.0"
+                 izz="0.000180"/>
+      </inertial>
     </link>
     <joint name="mid360_mount_joint" type="fixed">
@@ -76,4 +86,42 @@
       <selfCollide>false</selfCollide>
     </gazebo>
+    <!-- Fortress gpu_lidar at the optical origin. Publishes LaserScan on
+         /livox/scan and PointCloudPacked on /livox/scan/points; sim_world
+         remaps the cloud to /livox/lidar. No per-point times, so consumers
+         must keep deskewed=false. IMU is not simulated (real /livox/imu
+         accelerations are in g). -->
+    <gazebo reference="mid360_mount_frame">
+      <gravity>false</gravity>
+      <selfCollide>false</selfCollide>
+      <sensor name="mid360s" type="gpu_lidar">
+        <always_on>true</always_on>
+        <update_rate>${livox_sim_update_hz}</update_rate>
+        <visualize>false</visualize>
+        <topic>livox/scan</topic>
+        <gz_frame_id>livox_frame</gz_frame_id>
+        <pose>${livox_optical_xyz} ${livox_optical_rpy}</pose>
+        <lidar>
+          <scan>
+            <horizontal>
+              <samples>${livox_sim_h_samples}</samples>
+              <resolution>1</resolution>
+              <min_angle>${livox_sim_h_min}</min_angle>
+              <max_angle>${livox_sim_h_max}</max_angle>
+            </horizontal>
+            <vertical>
+              <samples>${livox_sim_v_samples}</samples>
+              <resolution>1</resolution>
+              <min_angle>${livox_sim_v_min}</min_angle>
+              <max_angle>${livox_sim_v_max}</max_angle>
+            </vertical>
+          </scan>
+          <range>
+            <min>${livox_sim_range_min}</min>
+            <max>${livox_sim_range_max}</max>
+            <resolution>0.01</resolution>
+          </range>
+        </lidar>
+      </sensor>
+    </gazebo>
   </xacro:macro>
 </robot>
