Commit message: feat(description): freeze D555 Layer 3 and Livox mount, add scene markers
Transplanted from origin/ros2_humble d88807a; scene_hardware was adapted to the local always-wall-time launch contract.

File: src/luggage_description/config/backups/20260911_2109_livox_d555_icp/mid360_origin.xacro (robot description, xacro)
@@ -1,4 +1,3 @@
 <?xml version="1.0"?>
-<!-- mid360_mount from D555-referenced ICP 2026-09-11, mount xyz 0.01 0.13 0.015 m. Camera Layer 3 is the reference. livox_optical/IMU stay handbook. CAD pad was 0.022 0.103 0.038 / 0 pi/2 pi/2. -->
 <!-- Mid-360S frames (Livox Mid-360 / Mid-360S user manual).
      livox_frame (point-cloud / ROS header):
@@ -17,6 +16,6 @@
        mount Z from the plate (handbook). -->
 <robot xmlns:xacro="http://www.ros.org/wiki/xacro">
-  <xacro:property name="mid360_mount_xyz" value="0.010000 0.130000 0.015000"/>
-  <xacro:property name="mid360_mount_rpy" value="0.16221799 1.63740799 1.77427038"/>
+  <xacro:property name="mid360_mount_xyz" value="0.022 0.103 0.038"/>
+  <xacro:property name="mid360_mount_rpy" value="0 1.57079633 1.57079633"/>
   <!-- Base of the sensor -> livox_frame (optical / point-cloud origin). -->
   <xacro:property name="livox_optical_xyz" value="0.000 0.000 0.047"/>

File: src/luggage_description/config/camera_mount_origin.xacro (robot description, xacro)
@@ -1,7 +1,7 @@
 <?xml version="1.0"?>
-<!-- Saved by eof_mount_stack_tune_gui.py -->
+<!-- Layer 3 from CC600 ChArUco eye-in-hand 2026-09-11 poses 21-38 (TSAI/PARK/DANIILIDIS mean). Do not edit Layers 1-2. -->
 <robot xmlns:xacro="http://www.ros.org/wiki/xacro">
   <xacro:property name="cam_mount_parent" value="eef_mount_adapter"/>
-  <xacro:property name="cam_mount_xyz" value="0.013000 0.097000 -0.021000"/>
-  <xacro:property name="cam_mount_rpy" value="0.03769911 1.36345121 1.57079633"/>
+  <xacro:property name="cam_mount_xyz" value="-0.028833 0.107910 -0.077120"/>
+  <xacro:property name="cam_mount_rpy" value="-0.01784105 1.39066481 1.56765511"/>
 </robot>
