Commit message: feat(description): lock EEF TF tree and D555 167x42x48 mm housing
Canonical wrist chain is flange CAD, solved adapter, CAD Livox pocket,
handbook +47 mm, and re-expressed ChArUco Layer 3. Camera visual is the
D555 datasheet envelope, not a D435 90 mm box.

Co-authored-by: Cursor <cursoragent@cursor.com>

File: src/luggage_description/config/backups/20260914_livox_pocket_adapter/mid360_origin.xacro (robot description, xacro)
@@ -1,9 +1,4 @@
 <?xml version="1.0"?>
-<!-- 2026-09-14: elfin_base_link<-livox is planar full-table then balanced corners+edges XY ICP plus mean-z (revision 2026-09-14_xy_balanced_corners_edges). CAD square pocket seats livox on the mounter; this joint is solved so that chain realizes T_icp. Camera Layer 3 re-expressed so T_end_optical stays CC600. -->
-<!-- mid360_mount_frame is the CAD square pocket on the adapter mesh
-     (0.022 0.103 0.038 / 0 pi/2 pi/2). 2026-09-14: groove-to-livox is
-     this CAD seating. elfin_base_link<-livox is frozen table ICP
-     (balanced corners+edges + mean-z). eef_mount_adapter vs EOF is
-     solved to close both. Optical/IMU stay handbook. -->
+<!-- mid360_mount from D555-referenced ICP 2026-09-11, mount xyz 0.01 0.13 0.015 m. Camera Layer 3 is the reference. livox_optical/IMU stay handbook. CAD pad was 0.022 0.103 0.038 / 0 pi/2 pi/2. -->
 <!-- Mid-360S frames (Livox Mid-360 / Mid-360S user manual).
      livox_frame (point-cloud / ROS header):
@@ -22,6 +17,6 @@
        mount Z from the plate (handbook). -->
 <robot xmlns:xacro="http://www.ros.org/wiki/xacro">
-  <xacro:property name="mid360_mount_xyz" value="0.022000 0.103000 0.038000"/>
-  <xacro:property name="mid360_mount_rpy" value="0.00000000 1.57079633 1.57079633"/>
+  <xacro:property name="mid360_mount_xyz" value="0.010000 0.130000 0.015000"/>
+  <xacro:property name="mid360_mount_rpy" value="0.16221799 1.63740799 1.77427038"/>
   <!-- Base of the sensor -> livox_frame (optical / point-cloud origin). -->
   <xacro:property name="livox_optical_xyz" value="0.000 0.000 0.047"/>

File: src/luggage_description/config/backups/20260914_xy_full_edges_mean_z/mid360_origin.xacro (robot description, xacro)
@@ -1,8 +1,8 @@
 <?xml version="1.0"?>
-<!-- 2026-09-14: elfin_base_link<-livox is planar full-table then balanced corners+edges XY ICP plus mean-z (revision 2026-09-14_xy_balanced_corners_edges). CAD square pocket seats livox on the mounter; this joint is solved so that chain realizes T_icp. Camera Layer 3 re-expressed so T_end_optical stays CC600. -->
+<!-- 2026-09-14: elfin_base_link<-livox is planar full-table + edges XY ICP plus mean-z (revision 2026-09-14_xy_full_edges_mean_z). CAD square pocket seats livox on the mounter; this joint is solved so that chain realizes T_icp. Camera Layer 3 re-expressed so T_end_optical stays CC600. -->
 <!-- mid360_mount_frame is the CAD square pocket on the adapter mesh
      (0.022 0.103 0.038 / 0 pi/2 pi/2). 2026-09-14: groove-to-livox is
      this CAD seating. elfin_base_link<-livox is frozen table ICP
-     (balanced corners+edges + mean-z). eef_mount_adapter vs EOF is
+     (xy full-table + edges + mean-z). eef_mount_adapter vs EOF is
      solved to close both. Optical/IMU stay handbook. -->
 <!-- Mid-360S frames (Livox Mid-360 / Mid-360S user manual).

File: src/luggage_description/config/camera_mount_origin.xacro (robot description, xacro)
@@ -1,7 +1,7 @@
 <?xml version="1.0"?>
-<!-- Layer 3 from CC600 ChArUco eye-in-hand 2026-09-11 poses 21-38 (TSAI/PARK/DANIILIDIS mean). Do not edit Layers 1-2. -->
+<!-- Layer 3 from CC600 ChArUco eye-in-hand 2026-09-11 poses 21-38 (TSAI/PARK/DANIILIDIS mean), re-expressed 2026-09-14 after seating CAD Mid-360 pocket under T_icp livox (revision 2026-09-14_xy_balanced_corners_edges). T_end_optical unchanged. Do not edit Layers 1-2. -->
 <robot xmlns:xacro="http://www.ros.org/wiki/xacro">
   <xacro:property name="cam_mount_parent" value="eef_mount_adapter"/>
-  <xacro:property name="cam_mount_xyz" value="-0.028833 0.107910 -0.077120"/>
-  <xacro:property name="cam_mount_rpy" value="-0.01784105 1.39066481 1.56765511"/>
+  <xacro:property name="cam_mount_xyz" value="-0.023249 0.099580 -0.052059"/>
+  <xacro:property name="cam_mount_rpy" value="0.02901151 1.32524323 1.59953586"/>
 </robot>

File: src/luggage_description/config/eef_mount_adapter_origin.xacro (robot description, xacro)
@@ -1,7 +1,7 @@
 <?xml version="1.0"?>
-<!-- Saved by eof_mount_stack_tune_gui.py -->
+<!-- 2026-09-14: elfin_base_link<-livox is planar full-table then balanced corners+edges XY ICP plus mean-z (revision 2026-09-14_xy_balanced_corners_edges). CAD square pocket seats livox on the mounter; this joint is solved so that chain realizes T_icp. Camera Layer 3 re-expressed so T_end_optical stays CC600. -->
 <robot xmlns:xacro="http://www.ros.org/wiki/xacro">
   <xacro:property name="adapter_mount_parent" value="suction_panel"/>
-  <xacro:property name="adapter_mount_xyz" value="0.016800 -0.015600 0.070200"/>
-  <xacro:property name="adapter_mount_rpy" value="1.57707939 -0.00003948 -3.13530959"/>
+  <xacro:property name="adapter_mount_xyz" value="0.021734 -0.033926 0.082591"/>
+  <xacro:property name="adapter_mount_rpy" value="1.51187936 -0.01424906 3.13751341"/>
 </robot>

File: src/luggage_description/urdf/eef_sensor_mount.urdf.xacro (robot description, xacro)
@@ -2,7 +2,8 @@
 <robot xmlns:xacro="http://www.ros.org/wiki/xacro" name="eef_sensor_mount">
   <!--
-    3D-printed sensor mount adapter that bolts onto elfin_link6 (EOF).
-    Hosts the RealSense D435 camera and the Mid-360S lidar frames.
+    3D-printed sensor mount adapter on suction_panel (EOF flange CAD).
+    Hosts the RealSense D555 PoE and the Mid-360S lidar frames.
     STL is in millimetres; scale 0.001 converts to metres for URDF.
+    Canonical joints: docs/architecture/eef_sensor_frames.md.
   -->
   <xacro:include filename="$(find luggage_description)/config/mid360_origin.xacro"/>
@@ -41,6 +42,6 @@
     </joint>
     <!-- Mid-360S: mechanical mount plus optical and IMU frames.
-         Origins come from config/mid360_origin.xacro (handbook optical/IMU;
-         xyz/rpy are the camera-tower +Y pad, not jointly calibrated). -->
+         Origins come from config/mid360_origin.xacro (CAD square pocket on
+         the +Y face of arm_realsense_v1.3; handbook optical/IMU). -->
     <link name="mid360_mount_frame">
       <!-- Housing 65 x 65 x 60 mm, origin at base centre, +Z through the dome.

File: src/luggage_description/urdf/realsense_d435.urdf.xacro (robot description, xacro)
@@ -2,22 +2,23 @@
 <robot xmlns:xacro="http://www.ros.org/wiki/xacro" name="realsense_d435">
   <!--
-    Intel RealSense D435 nominal frame convention:
-      camera_link +X = depth/camera forward
-      camera_link +Y = 90 mm long axis / stereo baseline axis
-      camera_link +Z = 25 mm height axis
-    Dimensions/extrinsics follow realsense2_description _d435.urdf.xacro.
-    Observe pose (world): optical +Z ~ [0,0,-1], camera +Y horizontal.
+    Hardware is D555 PoE in a D555-sized printed pocket (not a D435 90 mm
+    pocket). camera_link +X = forward; +Y = stereo baseline / long axis;
+    +Z = height. Visual/collision use D555 Datasheet v1.1 envelope
+    167 x 42 x 48 mm (L x H x D). camera_link is left IR (d555_link identity).
+    Front face at camera_link +X = 0; body extends -X into the mount.
+    Y offset 47.5 mm is half of the 95 mm stereo baseline.
+    cam_mount_* (ChArUco Layer 3) is the optical/body pose and is not this box.
   -->
   <xacro:macro name="realsense_d435" params="parent *origin depth_near:=0.105 depth_far:=3.0">
     <xacro:property name="d435_cam_depth_to_color_offset" value="0.015"/>
-    <xacro:property name="d435_cam_depth" value="0.02505"/>
-    <xacro:property name="d435_cam_width" value="0.090"/>
-    <xacro:property name="d435_cam_height" value="0.025"/>
-    <xacro:property name="d435_cam_depth_py" value="0.0175"/>
+    <xacro:property name="d555_cam_depth" value="0.048"/>
+    <xacro:property name="d555_cam_length" value="0.167"/>
+    <xacro:property name="d555_cam_height" value="0.042"/>
+    <xacro:property name="d555_cam_py" value="0.0475"/>
     <link name="camera_link">
       <visual>
-        <origin xyz="0 ${-d435_cam_depth_py} 0" rpy="0 0 0"/>
+        <origin xyz="${-d555_cam_depth/2} ${-d555_cam_py} 0" rpy="0 0 0"/>
         <geometry>
-          <box size="${d435_cam_depth} ${d435_cam_width} ${d435_cam_height}"/>
+          <box size="${d555_cam_depth} ${d555_cam_length} ${d555_cam_height}"/>
         </geometry>
         <material name="camera_grey">
@@ -25,9 +26,9 @@
         </material>
       </visual>
-      <!-- Lens/front marker on +X face (90 x 25 mm), matching official camera_link +X forward. -->
+      <!-- Lens/front marker on +X face (167 x ~42 mm). -->
       <visual name="camera_lens_marker">
-        <origin xyz="0.013025 ${-d435_cam_depth_py} 0" rpy="0 0 0"/>
+        <origin xyz="0.0005 ${-d555_cam_py} 0" rpy="0 0 0"/>
         <geometry>
-          <box size="0.001 0.09 0.022"/>
+          <box size="0.001 ${d555_cam_length} 0.038"/>
         </geometry>
         <material name="camera_lens_dark">
@@ -36,12 +37,12 @@
       </visual>
       <collision>
-        <origin xyz="0 ${-d435_cam_depth_py} 0" rpy="0 0 0"/>
+        <origin xyz="${-d555_cam_depth/2} ${-d555_cam_py} 0" rpy="0 0 0"/>
         <geometry>
-          <box size="${d435_cam_depth} ${d435_cam_width} ${d435_cam_height}"/>
+          <box size="${d555_cam_depth} ${d555_cam_length} ${d555_cam_height}"/>
         </geometry>
       </collision>
       <inertial>
-        <!-- Intel's URDF notes these inertias are nominal visual-model values. -->
-        <mass value="0.072"/>
+        <!-- D555 datasheet mass is 337 g; tensor is still a nominal visual-model value. -->
+        <mass value="0.337"/>
         <inertia ixx="0.003881243" ixy="0.0" ixz="0.0"
                  iyy="0.000498940" iyz="0.0"
@@ -54,7 +55,7 @@
       <xacro:insert_block name="origin"/>
     </joint>
-    <!-- D555 (PoE) sits in the same printed pocket as this D435. Body pose
-         is camera_link (cam_mount_*). Driver publishes d555_* optical frames
-         from d555_link; do not duplicate those here. -->
+    <!-- D555 (PoE) in the printed D555 pocket. Body pose is camera_link
+         (cam_mount_*, ChArUco Layer 3). Driver publishes d555_* optical
+         frames from d555_link; do not duplicate those here. -->
     <link name="d555_link"/>
     <joint name="d555_body_joint" type="fixed">
